File: board/board.kicad_pcb (KiCad board)
At the start: 2 copper layers, 21 x 13 mm, 1 part

Commit message: initial
Parts:
- added C1: 2.2uF, Capacitor_SMD:C_1210_3225Metric, F.Cu at (146.3, 94.6)
- added C10: 4.7nF, Capacitor_SMD:C_0603_1608Metric, F.Cu at (162.7, 99.9)
- added C2: 2.2uF, Capacitor_SMD:C_1210_3225Metric, F.Cu at (149.6, 94.6)
- added C3: 2.2uF, Capacitor_SMD:C_1210_3225Metric, F.Cu at (152.8, 94.6)
- added C4: 2.2uF, Capacitor_SMD:C_1210_3225Metric, F.Cu at (156.7, 95.5)
- added C5: 100nF, Capacitor_SMD:C_0603_1608Metric, F.Cu at (161.2, 96.2)
- added C6: 47uF, Capacitor_SMD:C_0805_2012Metric, F.Cu at (162.6, 91.8)
- added C7: 47uF, Capacitor_SMD:C_0805_2012Metric, F.Cu at (158.6, 91.8)
- added C8: 47uF, Capacitor_SMD:C_0805_2012Metric, F.Cu at (160.6, 91.8)
- added C9: 47pF, Capacitor_SMD:C_0603_1608Metric, F.Cu at (161.2, 99.9)
- added D1: D560C, Diode_SMD:D_SMC, F.Cu at (166.8, 97.0)
- added J1: 003_power, on_edge:on_edge_2x05_host, F.Cu at (185.0, 96.5)
- added J2: 013_PoE_rectified, on_edge:on_edge_2x05_device, F.Cu at (140.0, 96.5)
- added L1: 6.8uH, Inductor_SMD:L_10.4x10.4_H4.8, F.Cu at (175.6, 96.2)
- added R1: 53.6k, Resistor_SMD:R_0603_1608Metric, F.Cu at (156.0, 90.9)
- added R2: 10.2k, Resistor_SMD:R_0603_1608Metric, F.Cu at (153.0, 90.9)
- added R3: 10k, Resistor_SMD:R_0603_1608Metric, F.Cu at (152.2, 101.1)
- added R4: 10k, Resistor_SMD:R_0603_1608Metric, F.Cu at (149.2, 101.1)
- added R5: 16.9k, Resistor_SMD:R_0603_1608Metric, F.Cu at (161.9, 102.2)
- added R6: 243k, Resistor_SMD:R_0603_1608Metric, F.Cu at (150.8, 101.1)
- added U1: TPS54560BDDA, Package_SO:Texas_R-PDSO-G8_EP2.95x4.9mm_Mask2.4x3.1mm_ThermalVias, F.Cu at (156.7, 99.9)
- LOGO1: moved to B.Cu
- moved LOGO1 23.3 mm to (173.2, 96.5), turned to 180 degrees
Routing:
- net GND: track 0.00 -> 61.0 mm, vias 0 -> 32
- net /step-down/5V: track 0.00 -> 31.4 mm, vias 0 -> 1
- net /step-down/fb: track 0.00 -> 28.5 mm, vias 0 -> 2
- net /step-down/48V: track 0.00 -> 26.9 mm
- net /step-down/sw: track 0.00 -> 18.1 mm
- net /step-down/boot: track 0.00 -> 8.07 mm, vias 0 -> 2
- net Net-(U1-EN): track 0.00 -> 6.92 mm
- net Net-(U1-RT/CLK): track 0.00 -> 4.02 mm
- net Net-(U1-COMP): track 0.00 -> 3.43 mm
- net Net-(C10-Pad1): track 0.00 -> 1.48 mm
- added copper zone on B.Cu, net GND
- added copper zone on F.Cu, net GND
Other:
- board size 21 x 13 mm -> 45 x 13 mm
